File: ise_sensor.kicad_sch (KiCad schematic)
At the start: 34 parts, among them U12 ADS122C04IRTER, U14 OPA928, U16 TPS7A2025PDBVR, U17 LM2776, U18 TPS72325DBV, U5 ADM3260

Commit message: Updates
Parts:
- added C49, C57: 100nF, Capacitor_SMD:C_0402_1005Metric, symbol Device:C_Small
- added C51: 10uF, Capacitor_SMD:C_0402_1005Metric, symbol Device:C_Small
- added C53: 50uF, Capacitor_SMD:C_0402_1005Metric, symbol Device:C_Small
- added C55, C56: 1uF, Capacitor_SMD:C_0402_1005Metric, symbol Device:C_Small
- added U1: REF5025IDR, EasyEDA:SOIC-8_L4.9-W3.9-P1.27-LS6.0-BL, symbol EasyEDA:REF5025IDR
Connections:
- net ISE_GND: now also C49.2, C51.2, C53.1, C55.1, C56.1, C57.2, U1.4 (GND); no longer U12.3 (AVSS)
- net TEMP: now reaches U12.5 (AIN2)
- net TEMP: now also U1.3 (TEMP)
- net ISO_-2V5 renamed PP_ISO_NEG_2V5
- net PP_ISO_NEG_2V5: now also U12.3 (AVSS), C49.1; no longer U12.6 (REFN)
- net ISO_-3V3 renamed PP_ISO_NEG_3V3
- net ISO_2V5 renamed PP_ISO_2V5
- net PP_ISO_2V5: now also C50.1, U12.10 (AVDD); no longer U12.7 (REFP)
- net ISO_3V3 renamed PP_ISO_3V3
- net PP_ISO_3V3: now also C51.1, U1.2 (VIN); no longer C50.1, U12.10 (AVDD)
- new net: C55.2, U1.5 (TRIM/NR)
- new net PP_ISO_REF_2V5: C53.2, C56.2, C57.1, U1.6 (VOUT), U12.7 (REFP)
- no-connect marks 5 -> 8
Other:
- note added: "2.5V Reference"
- note added: "ADC"
- note added: "I2C"
- note added: "ISE Sensor Buffer"
- note added: "Isolation"
- note added: "Power"
- note removed: "POWER"
- moved on the sheet: C18, C19, C20, C21, C22, C23, C24, C25, C34, C35, C36, C37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
